File: luaos.kicad_pcb (KiCad board)
At the start: 2 copper layers, 102.8 x 66 mm, 21 parts, among them J1 Screw_Terminal_01x02, J10 Conn_1, J11 Conn_1, J12 Conn_01x02_Socket, J13 Conn_01x08_Socket, J14 Conn_01x05_Socket, J2 Conn_01x03, J3 Conn_01x05_Socket, J4 Conn_01x08_Socket, J5 HLK-PM1, J6 Conn_01x03_Socket, J7 Conn_01x03_Socket, J8 Conn_2, J9 Conn_2, U1 ESP32-C3_Luaos, U2 siwi_D1_mini_Fassung, U3 siwi_D1_mini_Fassung

Commit message: Version 0.2 neues PCB Design
Parts:
- removed J10, J11: Conn_1, Connector_PinHeader_2.54mm:PinHeader_1x08_P2.54mm_Vertical
- removed J13: Conn_01x08_Socket, Connector_PinHeader_2.54mm:PinHeader_1x08_P2.54mm_Vertical
- removed J14: Conn_01x05_Socket, Connector_PinHeader_2.54mm:PinHeader_1x05_P2.54mm_Vertical
- added J15: Conn_1, Connector_PinHeader_2.54mm:PinHeader_1x08_P2.54mm_Vertical, F.Cu at (146.9, 78.3)
- added J16: Conn_1, Connector_PinHeader_2.54mm:PinHeader_1x08_P2.54mm_Vertical, F.Cu at (146.9, 134.2)
- added J17: Screw_Terminal_01x02, TerminalBlock:TerminalBlock_MaiXu_MX126-5.0-02P_1x02_P5.00mm, F.Cu at (170.4, 116.3)
- added J18: Screw_Terminal_01x02, TerminalBlock:TerminalBlock_MaiXu_MX126-5.0-02P_1x02_P5.00mm, F.Cu at (171.0, 95.9)
- added J19: Screw_Terminal_01x01, TerminalBlock_MetzConnect:TerminalBlock_MetzConnect_360271_1x01_Horizontal_ScrewM3.0_Boxed, F.Cu at (171.0, 83.8)
- added J20: Screw_Terminal_01x02, siwi_Footprints:siwi_Converter_ACDC_HLK-5Mxx_230V, F.Cu at (199.4, 88.4)
- added J21: Screw_Terminal_01x02, TerminalBlock:TerminalBlock_MaiXu_MX126-5.0-02P_1x02_P5.00mm, F.Cu at (188.0, 88.9)
- added Q1: IRLZ44N, Package_TO_SOT_THT:TO-220-3_Vertical, F.Cu at (197.6, 130.9)
- added Q2: IRLZ44N, Package_TO_SOT_THT:TO-220-3_Vertical, F.Cu at (191.9, 125.8)
- added R1: R, siwi_Footprints:siwi_R_Axial_DIN0204_L3.6mm_D1.6mm_P7.62mm_Horizontal, F.Cu at (149.9, 90.8)
- added R2: R, siwi_Footprints:siwi_R_Axial_DIN0204_L3.6mm_D1.6mm_P7.62mm_Horizontal, F.Cu at (146.9, 93.3)
- added R3: R, siwi_Footprints:siwi_R_Axial_DIN0204_L3.6mm_D1.6mm_P7.62mm_Horizontal, F.Cu at (146.7, 118.7)
- added R4: R, siwi_Footprints:siwi_R_Axial_DIN0204_L3.6mm_D1.6mm_P7.62mm_Horizontal, F.Cu at (149.2, 128.9)
- added R5: R, siwi_Footprints:siwi_R_Axial_DIN0204_L3.6mm_D1.6mm_P7.62mm_Horizontal, F.Cu at (183.0, 123.9)
- added R6: R, siwi_Footprints:siwi_R_Axial_DIN0204_L3.6mm_D1.6mm_P7.62mm_Horizontal, F.Cu at (186.2, 120.7)
- added REF**: MountingHole_4.3mm_M4, MountingHole:MountingHole_4.3mm_M4, F.Cu at (186.7, 105.4)
- added REF**: MountingHole_4.3mm_M4, MountingHole:MountingHole_4.3mm_M4, F.Cu at (186.1, 77.5)
- added U4: PC817, siwi_Footprints:siwi_PC4SF, F.Cu at (153.2, 90.8)
- added U5: PC817, siwi_Footprints:siwi_PC4SF, F.Cu at (153.2, 101.0)
- added U6: PC817, siwi_Footprints:siwi_PC4SF, F.Cu at (153.2, 111.1)
- added U7: PC817, siwi_Footprints:siwi_PC4SF, F.Cu at (153.2, 121.3)
- J1: value Screw_Terminal_01x02 -> Conn_1; footprint TerminalBlock:TerminalBlock_MaiXu_MX126-5.0-02P_1x02_P5.00mm -> Connector_PinHeader_2.54mm:PinHeader_1x08_P2.54mm_Vertical
- J12: footprint Connector_PinHeader_1.00mm:PinHeader_1x02_P1.00mm_Vertical -> Connector_PinHeader_2.54mm:PinHeader_1x02_P2.54mm_Vertical
- J2: value Conn_01x03 -> Conn_01x03_Socket
- J3: value Conn_01x05_Socket -> Conn_1; footprint Connector_PinHeader_2.54mm:PinHeader_1x05_P2.54mm_Vertical -> Connector_PinHeader_2.54mm:PinHeader_1x08_P2.54mm_Vertical
- J4: value Conn_01x08_Socket -> Screw_Terminal_01x03; footprint Connector_PinHeader_2.54mm:PinHeader_1x08_P2.54mm_Vertical -> TerminalBlock:TerminalBlock_bornier-3_P5.08mm
- J5: footprint Library:Converter_ACDC_Hi-Link_HLK-PMxx -> siwi_Footprints:siwi_HLK-PMxx_DC
- J8: value Conn_2 -> Conn_01x20_Socket; footprint Connector_PinHeader_2.54mm:PinHeader_1x08_P2.54mm_Vertical -> siwi_Footprints:siwi_PinHeader_2x20_P2.54
- J9: value Conn_2 -> Conn_01x03_Socket; footprint Connector_PinHeader_2.54mm:PinHeader_1x08_P2.54mm_Vertical -> Connector_PinHeader_2.54mm:PinHeader_1x03_P2.54mm_Vertical
- U1: footprint Library:ESP32-C3-luaos -> siwi_Footprints:siwi_ESP32-C3-luaos
- U2, U3: footprint Library:siwi_WEMOS_D1_mini_light -> siwi_Footprints:siwi_D1_mini_steckplatz
- moved J1 136.7 mm to (185.5, 113.1), turned to 90 degrees
- moved J4 119.9 mm to (205.3, 130.2), turned to 90 degrees
- moved REF** 95.4 mm to (136.0, 79.0)
- moved J3 94.9 mm to (185.5, 136.0), turned to 90 degrees
- moved REF** 74.7 mm to (48.0, 79.0)
- moved J9 71.8 mm to (63.5, 113.7), turned to 0 degrees
- moved REF** 47.7 mm to (136.0, 132.0)
- moved J8 40.7 mm to (94.6, 85.3), turned to 0 degrees
- moved REF** 29.6 mm to (48.0, 132.0)
- moved J2 16.3 mm to (81.3, 132.7), turned to 90 degrees
- moved J5 13.5 mm to (48.3, 106.8)
- moved U3 6.63 mm to (111.1, 133.9)
- moved U2 6.29 mm to (111.1, 100.9)
- moved J12 2.62 mm to (113.7, 106.0)
- moved J6 2.54 mm to (63.5, 102.9)
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Connections:
- J1 pad 1: GND -> Net-(J1-Pin_1)
- J1 pad 2: +5V -> unconnected-(J1-Pin_2-Pad2)
- J2 pad 1: +3.3V -> GND
- J2 pad 3: GND -> +3.3V
- J3 pad 1: +3.3V -> unconnected-(J3-Pin_1-Pad1)
- J3 pad 2: GND -> unconnected-(J3-Pin_2-Pad2)
- J3 pad 3: Net-(J14-Pin_3) -> unconnected-(J3-Pin_3-Pad3)
- J3 pad 4: Net-(J14-Pin_4) -> unconnected-(J3-Pin_4-Pad4)
- J3 pad 5: Net-(J14-Pin_5) -> unconnected-(J3-Pin_5-Pad5)
- J4 pad 1: +3.3V -> Net-(J4-Pin_1)
- J4 pad 2: GND -> Net-(J4-Pin_2)
- J4 pad 3: Net-(J13-Pin_3) -> Net-(J1-Pin_7)
- J5 pad 1: +5V -> GND
- J5 pad 2: GND -> +5V
- J8 pad 1: +5V -> +3.3V
- J9 pad 1: +5V -> Net-(J9-Pin_1)
- U1 pad 10: Net-(J8-Pin_6) -> Net-(U1-GPIO13)
- U1 pad 12: unconnected-(U1-REST-Pad12) -> Net-(J9-Pin_1)
- U1 pad 15: unconnected-(U1-PWB-Pad15) -> Net-(J9-Pin_3)
- U1 pad 19: Net-(J13-Pin_4) -> Net-(J8-Pin_4)
- U1 pad 20: Net-(J13-Pin_3) -> Net-(J8-Pin_3)
- U1 pad 21: Net-(J13-Pin_5) -> Net-(J8-Pin_5)
- U1 pad 22: Net-(J13-Pin_7) -> Net-(J8-Pin_7)
- U1 pad 23: Net-(J13-Pin_6) -> Net-(J8-Pin_6)
- U1 pad 24: Net-(J13-Pin_8) -> Net-(J8-Pin_9)
- U1 pad 27: Net-(J14-Pin_3) -> Net-(J8-Pin_12)
- U1 pad 28: Net-(J14-Pin_4) -> Net-(J8-Pin_13)
- U1 pad 29: unconnected-(U1-GPIO8-Pad29) -> Net-(J8-Pin_8)
- U1 pad 30: Net-(J14-Pin_5) -> Net-(J8-Pin_14)
- U1 pad 5: unconnected-(U1-GPIO18-Pad5) -> Net-(J8-Pin_15)
- U1 pad 6: unconnected-(U1-GPIO19-Pad6) -> Net-(J8-Pin_16)
- U2 pad 1: Net-(J10-Pin_1) -> unconnected-(U2-~{RST}-Pad1)
- U2 pad 11: Net-(J8-Pin_3) -> unconnected-(U2-D4-Pad11)
- U2 pad 12: Net-(J8-Pin_4) -> unconnected-(U2-D3-Pad12)
- U2 pad 13: Net-(J8-Pin_5) -> unconnected-(U2-SDA/D2-Pad13)
- U2 pad 14: Net-(J8-Pin_6) -> Net-(U1-GPIO13)
- U2 pad 15: Net-(J8-Pin_7) -> unconnected-(U2-RX-Pad15)
- U2 pad 16: Net-(J8-Pin_8) -> unconnected-(U2-TX-Pad16)
- U2 pad 2: Net-(J10-Pin_2) -> unconnected-(U2-A0-Pad2)
- U2 pad 3: Net-(J10-Pin_3) -> unconnected-(U2-D0-Pad3)
- U2 pad 4: Net-(J10-Pin_4) -> unconnected-(U2-SCK/D5-Pad4)
- U2 pad 5: Net-(J10-Pin_5) -> unconnected-(U2-MISO/D6-Pad5)
- U2 pad 6: Net-(J10-Pin_6) -> unconnected-(U2-MOSI/D7-Pad6)
- U2 pad 7: Net-(J10-Pin_7) -> unconnected-(U2-CS/D8-Pad7)
- U3 pad 1: Net-(J11-Pin_1) -> unconnected-(U3-~{RST}-Pad1)
- U3 pad 11: Net-(J9-Pin_3) -> unconnected-(U3-D4-Pad11)
- U3 pad 12: Net-(J9-Pin_4) -> unconnected-(U3-D3-Pad12)
- U3 pad 13: Net-(J9-Pin_5) -> unconnected-(U3-SDA/D2-Pad13)
- U3 pad 15: Net-(J9-Pin_7) -> unconnected-(U3-RX-Pad15)
- U3 pad 16: Net-(J9-Pin_8) -> unconnected-(U3-TX-Pad16)
- U3 pad 2: Net-(J11-Pin_2) -> unconnected-(U3-A0-Pad2)
- U3 pad 3: Net-(J11-Pin_3) -> unconnected-(U3-D0-Pad3)
- U3 pad 4: Net-(J11-Pin_4) -> unconnected-(U3-SCK/D5-Pad4)
- U3 pad 5: Net-(J11-Pin_5) -> unconnected-(U3-MISO/D6-Pad5)
- U3 pad 6: Net-(J11-Pin_6) -> unconnected-(U3-MOSI/D7-Pad6)
- U3 pad 7: Net-(J11-Pin_7) -> unconnected-(U3-CS/D8-Pad7)
Routing:
- net Net-(J7-Pin_3): track 6.43 -> 128.2 mm, vias 0 -> 1
- net Net-(U1-GPIO13): track 0.00 -> 118.9 mm
- net Net-(J8-Pin_6): track 120.9 -> 14.8 mm
- net Net-(J19-Pin_1): track 0.00 -> 76.0 mm
- net Net-(J8-Pin_16): track 0.00 -> 64.1 mm
- net Net-(J8-Pin_15): track 0.00 -> 62.4 mm
- net Net-(J15-Pin_7): track 0.00 -> 60.6 mm
- net +5V: track 239.4 -> 195.6 mm
- net Net-(J1-Pin_7): track 0.00 -> 27.6 mm
- net Net-(J8-Pin_8): track 5.10 -> 23.5 mm
- net Net-(J13-Pin_3): track 15.6 -> 0.00 mm
- net Net-(J13-Pin_6): track 15.6 -> 0.00 mm
- net Net-(J16-Pin_1): track 0.00 -> 15.5 mm
- net GND: track 59.9 -> 44.8 mm
- net Net-(J15-Pin_1): track 0.00 -> 15.1 mm
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- added copper zone on B.Cu, net GND
Other:
- board size 102.8 x 66 mm -> 168 x 66.6 mm
- board text added: "1"
- board text added: "11"
- board text added: "12"
- board text added: "13"
- board text added: "14"
- board text added: "15"
- board text added: "16"
- board text added: "2"
- board text added: "230 V"
- board text added: "3"
- board text added: "4"
- board text added: "5"
- board text added: "5V"
- board text added: "6"
- board text added: "7"
- board text added: "CLK"
- board text added: "EN"
- board text added: "ESP32Lua V0.2"
- board text added: "GP0"
- board text added: "GP08"
- board text added: "GP09"
- board text added: "GP18"
- board text added: "GP19"
- board text added: "N"
- board text added: "P1"
- board text added: "P2"
- board text added: "P3"
- board text added: "P4"
- board text added: "PWB"
- board text added: "S21ME8"
- board text added: "SCL"
- board text added: "SDA"
- board text added: "U4"
- board text removed: "ESP32 Lua V 0.1"
- board text removed: "SPI_CK"
