File: luaos.kicad_sch (KiCad schematic)
At the start: 17 parts, among them J1 Screw_Terminal_01x02, J10 Conn_1, J11 Conn_1, J12 Conn_01x02_Socket, J13 Conn_01x08_Socket, J14 Conn_01x05_Socket, J2 Conn_01x03, J3 Conn_01x05_Socket, J4 Conn_01x08_Socket, J5 HLK-PM1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

Commit message: Version 0.2 neues PCB Design
Parts:
- removed J1: Screw_Terminal_01x02, TerminalBlock:TerminalBlock_MaiXu_MX126-5.0-02P_1x02_P5.00mm, symbol Connector:Screw_Terminal_01x02
- removed J10, J11: Conn_1, Connector_PinHeader_2.54mm:PinHeader_1x08_P2.54mm_Vertical, symbol Connector:Conn_01x08_Socket
- removed J13, J4: Conn_01x08_Socket, Connector_PinHeader_2.54mm:PinHeader_1x08_P2.54mm_Vertical, symbol Connector:Conn_01x08_Socket
- removed J14, J3: Conn_01x05_Socket, Connector_PinHeader_2.54mm:PinHeader_1x05_P2.54mm_Vertical, symbol Connector:Conn_01x05_Socket
- removed J2: Conn_01x03, Connector_PinHeader_2.54mm:PinHeader_1x03_P2.54mm_Vertical, symbol Connector_Generic:Conn_01x03
- removed J8, J9: Conn_2, Connector_PinHeader_2.54mm:PinHeader_1x08_P2.54mm_Vertical, symbol Connector:Conn_01x08_Socket
- added J1, J15, J16, J3: Conn_1, Connector_PinHeader_2.54mm:PinHeader_1x08_P2.54mm_Vertical, symbol Connector:Conn_01x08_Socket
- added J17, J18, J21: Screw_Terminal_01x02, TerminalBlock:TerminalBlock_MaiXu_MX126-5.0-02P_1x02_P5.00mm, symbol Connector:Screw_Terminal_01x02
- added J19: Screw_Terminal_01x01, TerminalBlock_MetzConnect:TerminalBlock_MetzConnect_360271_1x01_Horizontal_ScrewM3.0_Boxed, symbol Connector:Screw_Terminal_01x01
- added J2, J9: Conn_01x03_Socket, Connector_PinHeader_2.54mm:PinHeader_1x03_P2.54mm_Vertical, symbol Connector:Conn_01x03_Socket
- added J20: Screw_Terminal_01x02, siwi_Footprints:siwi_Converter_ACDC_HLK-5Mxx_230V, symbol Connector:Screw_Terminal_01x02
- added J4: Screw_Terminal_01x03, TerminalBlock:TerminalBlock_bornier-3_P5.08mm, symbol Connector:Screw_Terminal_01x03
- added J8: Conn_01x20_Socket, siwi_Footprints:siwi_PinHeader_2x20_P2.54, symbol Connector:Conn_01x20_Socket
- added Q1, Q2: IRLZ44N, Package_TO_SOT_THT:TO-220-3_Vertical, symbol Transistor_FET:IRLZ44N
- added R1, R2, R3, R4, R5, R6: R, siwi_Footprints:siwi_R_Axial_DIN0204_L3.6mm_D1.6mm_P7.62mm_Horizontal, symbol Device:R
- added U4, U5, U6, U7: PC817, siwi_Footprints:siwi_PC4SF, symbol Isolator:PC817
- J12: footprint Connector_PinHeader_1.00mm:PinHeader_1x02_P1.00mm_Vertical -> Connector_PinHeader_2.54mm:PinHeader_1x02_P2.54mm_Vertical
- J5: footprint Library:Converter_ACDC_Hi-Link_HLK-PMxx -> siwi_Footprints:siwi_HLK-PMxx_DC
- U1: footprint ESP32-C3-luaos -> siwi_Footprints:siwi_ESP32-C3-luaos
- U2, U3: footprint Library:siwi_WEMOS_D1_mini_light -> siwi_Footprints:siwi_D1_mini_steckplatz
Connections:
- net +3.3V: now also J2.3 (Pin_3), J8.1 (Pin_1), J8.10 (Pin_10), J8.20 (Pin_20)
- net +5V: now also J5.2 (Pin_2); no longer J5.1 (Pin_1)
- net GND: now also J5.1 (Pin_1), J2.1 (Pin_1), J8.11 (Pin_11), J8.18 (Pin_18), J8.2 (Pin_2), J9.2 (Pin_2); no longer J5.2 (Pin_2)
- net at J7.2 (Pin_2), U1.2 (GPIO0): now also J2.2 (Pin_2), J8.19 (Pin_19)
- net at U1.20 (SPI_MOSI): now also J8.3 (Pin_3)
- net at U1.19 (SPI_CK): now also J8.4 (Pin_4)
- net at U1.21 (SPI_MISO): now also J8.5 (Pin_5)
- net at U1.23 (GPIO7): now also J8.6 (Pin_6)
- net at U1.22 (GPIO6): now also J8.7 (Pin_7)
- net at U1.24 (GPIO11): now also J8.9 (Pin_9)
- net at U1.12 (REST): now also J9.1 (Pin_1)
- net at U1.15 (PWB): now also J9.3 (Pin_3)
- net at U1.27 (I2C_SCL): now also J8.12 (Pin_12)
- net at U1.28 (I2C_SDA): now also J8.13 (Pin_13)
- net at U1.29 (GPIO8): now also J8.8 (Pin_8)
- net at J7.3 (Pin_3), U1.3 (GPIO1): now also J8.17 (Pin_17)
- net at U1.30 (GPIO9): now also J8.14 (Pin_14)
- net at U1.5 (GPIO18): now also J8.15 (Pin_15)
- net at U1.6 (GPIO19): now also J8.16 (Pin_16)
- new net: Q1.1 (G), R5.2
- new net: J4.1 (Pin_1), Q1.2 (D)
- new net: J1.7 (Pin_7), J4.3 (Pin_3), Q1.3 (S), Q2.3 (S)
- new net: J15.1 (Pin_1), R2.1
- new net: J15.3 (Pin_3), R1.2
- new net: J15.7 (Pin_7), U4.2, U5.2, U6.2, U7.2
- new net: R3.2, U6.1
- new net: J19.1 (Pin_1), U4.3, U5.3, U6.3, U7.3
- new net: J17.1 (Pin_1), U6.4
- new net: J1.1 (Pin_1), R5.1
- new net: J1.3 (Pin_3), R6.1
- new net: R4.2, U7.1
- new net: J17.2 (Pin_2), U7.4
- new net: J16.2 (Pin_2), R4.1
- new net: R1.1, U4.1
- new net: J18.1 (Pin_1), U4.4
- new net: Q2.1 (G), R6.2
- new net: J4.2 (Pin_2), Q2.2 (D)
- new net: J20.1 (Pin_1), J21.1 (Pin_1)
- new net: J20.2 (Pin_2), J21.2 (Pin_2)
- new net: J16.1 (Pin_1), R3.1
- new net: J18.2 (Pin_2), U5.4
- new net: R2.2, U5.1
Other:
- moved on the sheet: J5
